File: esp32-led-matrix.kicad_sch (KiCad schematic)
At the start: 70 parts, among them J1 Conn_01x03, J2 Conn_01x03, J4 USB_C_Receptacle_USB2.0_16P, SW1 RESET, U1 ESP32-C6-WROOM-1-N8, U2 USBLC6-2SC6, U3 AMS1117-3.3(TO-252)

Commit message: process
Parts:
- removed D1, D2, D3, D4, D5, D6, D7, D8, D9: WS2812B, PCM_SparkFun-LED:WS2812_2020, symbol PCM_SparkFun-LED:WS2812B_2020
- removed D101: POWER, LED_SMD:LED_0603_1608Metric, symbol Device:LED_Small
- removed J1, J2: Conn_01x03, Connector_PinHeader_2.54mm:PinHeader_1x03_P2.54mm_Vertical, symbol Connector_Generic:Conn_01x03
- added D1: POWER, LED_SMD:LED_0603_1608Metric, symbol Device:LED_Small
- added D100, D101, D102, D103, D104, D105, D106, D107, D108, D109, D110, D111, D112, D113, D114, D115, D116, D117, D118, D119, D120, D121, D122, D123, D124, D125, D126, D127, D128, D129, D130, D131, D132, D133, D134, D135, D136, D137, D51, D52, D53, D54, D55, D56, D57, D58, D59, D60, D61, D62, D63, D64, D65, D66, D67, D68, D69, D70, D71, D72, D73, D74, D75, D76, D77, D78, D79, D80, D81, D82, D83, D84, D85, D86, D87, D88, D89, D90, D91, D92, D93, D94, D95, D96, D97, D98, D99: WS2812B, PCM_SparkFun-LED:WS2812_2020, symbol PCM_SparkFun-LED:WS2812B_2020
- added J2: Conn_01x04, PCM_SparkFun-Connector:JST_1x04_P2.0mm_Horizontal_SMD, symbol PCM_SparkFun-Connector:Conn_01x04_JST_P2.0mm_Horizontal_SMD
- D10, D11, D12, D13, D14, D15, D16, D17, D18, D19, D20, D21, D22, D23, D24, D25, D26, D27, D28, D29, D30, D31, D32, D33, D34, D35, D36, D37, D38, D39, D40, D41, D42, D43, D44, D45, D46, D47, D48, D49, D50: LCSC (none) -> C5349955; MPN (none) -> XL-2020RGBC-2812B
Connections:
- net GND is gone; now on net +5V: C1.2, C2.2, C3.2, C4.2, C5.2, C6.2, D4.1 (A1), J4.A1 (GND), J4.A12 (GND), J4.B1 (GND), J4.B12 (GND), J4.S1 (SHIELD), R1.2, R2.2, SW1.1 (A), U1.1 (GND), U1.28 (GND), U1.29 (GND), U2.2 (GND), U3.1 (GND)
- net +5V: now also D10.2 (VSS), D10.4 (VDD), D11.2 (VSS), D11.4 (VDD), D12.2 (VSS), D12.4 (VDD), D13.2 (VSS), D13.4 (VDD), D14.2 (VSS), D14.4 (VDD), D15.2 (VSS), D15.4 (VDD), D16.2 (VSS), D16.4 (VDD), D17.2 (VSS), D17.4 (VDD), D18.2 (VSS), D18.4 (VDD), D19.2 (VSS), D19.4 (VDD), D20.2 (VSS), D20.4 (VDD), D21.2 (VSS), D21.4 (VDD), D22.2 (VSS), D22.4 (VDD), D23.2 (VSS), D23.4 (VDD), D24.2 (VSS), D24.4 (VDD), D25.2 (VSS), D25.4 (VDD), D26.2 (VSS), D26.4 (VDD), D27.2 (VSS), D27.4 (VDD), D28.2 (VSS), D28.4 (VDD), D29.2 (VSS), D29.4 (VDD), D30.2 (VSS), D30.4 (VDD), D31.2 (VSS), D31.4 (VDD), D32.2 (VSS), D32.4 (VDD), D33.2 (VSS), D33.4 (VDD), D34.2 (VSS), D34.4 (VDD), D35.2 (VSS), D35.4 (VDD), D36.2 (VSS), D36.4 (VDD), D37.2 (VSS), D37.4 (VDD), D38.2 (VSS), D38.4 (VDD), D39.2 (VSS), D39.4 (VDD), D40.2 (VSS), D40.4 (VDD), D41.2 (VSS), D41.4 (VDD), D42.2 (VSS), D42.4 (VDD), D43.2 (VSS), D43.4 (VDD), D44.2 (VSS), D44.4 (VDD), D45.2 (VSS), D45.4 (VDD), D46.2 (VSS), D46.4 (VDD), D47.2 (VSS), D47.4 (VDD), D48.2 (VSS), D48.4 (VDD), D49.2 (VSS), D49.4 (VDD), D50.2 (VSS), D50.4 (VDD), D1.1 (K), D100.2 (VSS), D100.4 (VDD), D101.2 (VSS), D101.4 (VDD), D102.2 (VSS), D102.4 (VDD), D103.2 (VSS), D103.4 (VDD), D104.2 (VSS), D104.4 (VDD), D105.2 (VSS), D105.4 (VDD), D106.2 (VSS), D106.4 (VDD), D107.2 (VSS), D107.4 (VDD), D108.2 (VSS), D108.4 (VDD), D109.2 (VSS), D109.4 (VDD), D110.2 (VSS), D110.4 (VDD), D111.2 (VSS), D111.4 (VDD), D112.2 (VSS), D112.4 (VDD), D113.2 (VSS), D113.4 (VDD), D114.2 (VSS), D114.4 (VDD), D115.2 (VSS), D115.4 (VDD), D116.2 (VSS), D116.4 (VDD), D117.2 (VSS), D117.4 (VDD), D118.2 (VSS), D118.4 (VDD), D119.2 (VSS), D119.4 (VDD), D120.2 (VSS), D120.4 (VDD), D121.2 (VSS), D121.4 (VDD), D122.2 (VSS), D122.4 (VDD), D123.2 (VSS), D123.4 (VDD), D124.2 (VSS), D124.4 (VDD), D125.2 (VSS), D125.4 (VDD), D126.2 (VSS), D126.4 (VDD), D127.2 (VSS), D127.4 (VDD), D128.2 (VSS), D128.4 (VDD), D129.2 (VSS), D129.4 (VDD), D130.2 (VSS), D130.4 (VDD), D131.2 (VSS), D131.4 (VDD), D132.2 (VSS), D132.4 (VDD), D133.2 (VSS), D133.4 (VDD), D134.2 (VSS), D134.4 (VDD), D135.2 (VSS), D135.4 (VDD), D136.2 (VSS), D136.4 (VDD), D137.2 (VSS), D137.4 (VDD), D51.2 (VSS), D51.4 (VDD), D52.2 (VSS), D52.4 (VDD), D53.2 (VSS), D53.4 (VDD), D54.2 (VSS), D54.4 (VDD), D55.2 (VSS), D55.4 (VDD), D56.2 (VSS), D56.4 (VDD), D57.2 (VSS), D57.4 (VDD), D58.2 (VSS), D58.4 (VDD), D59.2 (VSS), D59.4 (VDD), D60.2 (VSS), D60.4 (VDD), D61.2 (VSS), D61.4 (VDD), D62.2 (VSS), D62.4 (VDD), D63.2 (VSS), D63.4 (VDD), D64.2 (VSS), D64.4 (VDD), D65.2 (VSS), D65.4 (VDD), D66.2 (VSS), D66.4 (VDD), D67.2 (VSS), D67.4 (VDD), D68.2 (VSS), D68.4 (VDD), D69.2 (VSS), D69.4 (VDD), D70.2 (VSS), D70.4 (VDD), D71.2 (VSS), D71.4 (VDD), D72.2 (VSS), D72.4 (VDD), D73.2 (VSS), D73.4 (VDD), D74.2 (VSS), D74.4 (VDD), D75.2 (VSS), D75.4 (VDD), D76.2 (VSS), D76.4 (VDD), D77.2 (VSS), D77.4 (VDD), D78.2 (VSS), D78.4 (VDD), D79.2 (VSS), D79.4 (VDD), D80.2 (VSS), D80.4 (VDD), D81.2 (VSS), D81.4 (VDD), D82.2 (VSS), D82.4 (VDD), D83.2 (VSS), D83.4 (VDD), D84.2 (VSS), D84.4 (VDD), D85.2 (VSS), D85.4 (VDD), D86.2 (VSS), D86.4 (VDD), D87.2 (VSS), D87.4 (VDD), D88.2 (VSS), D88.4 (VDD), D89.2 (VSS), D89.4 (VDD), D90.2 (VSS), D90.4 (VDD), D91.2 (VSS), D91.4 (VDD), D92.2 (VSS), D92.4 (VDD), D93.2 (VSS), D93.4 (VDD), D94.2 (VSS), D94.4 (VDD), D95.2 (VSS), D95.4 (VDD), D96.2 (VSS), D96.4 (VDD), D97.2 (VSS), D97.4 (VDD), D98.2 (VSS), D98.4 (VDD), D99.2 (VSS), D99.4 (VDD), J2.1, J2.4
- net Net-(D25-DOUT): now reaches D25.1 (DOUT)
- net Net-(D25-DOUT): now also D26.3 (DIN)
- net Net-(D24-DOUT): now reaches D24.1 (DOUT), D25.3 (DIN)
- net Net-(D50-DOUT): now reaches D50.1 (DOUT)
- net Net-(D50-DOUT): now also D51.3 (DIN)
- net Net-(D49-DOUT): now reaches D49.1 (DOUT), D50.3 (DIN)
- net Net-(D36-DOUT): now reaches D36.1 (DOUT), D37.3 (DIN)
- net Net-(D35-DOUT): now reaches D36.3 (DIN)
- net Net-(D35-DOUT): now also D35.1 (DOUT)
- net Net-(D14-DOUT): now reaches D14.1 (DOUT), D15.3 (DIN)
- net Net-(D13-DOUT): now reaches D13.1 (DOUT), D14.3 (DIN)
- net Net-(D30-DOUT): now reaches D30.1 (DOUT)
- net Net-(D30-DOUT): now also D31.3 (DIN)
- net Net-(D29-DOUT): now reaches D29.1 (DOUT), D30.3 (DIN)
- net Net-(D47-DOUT): now reaches D47.1 (DOUT), D48.3 (DIN)
- net Net-(D46-DOUT): now reaches D46.1 (DOUT), D47.3 (DIN)
- net Net-(D19-DOUT): now reaches D19.1 (DOUT), D20.3 (DIN)
- net Net-(D18-DOUT): now reaches D18.1 (DOUT), D19.3 (DIN)
- net at R3.2: now also D1.2 (A)
- net Net-(D11-DOUT): now reaches D11.1 (DOUT), D12.3 (DIN)
- net Net-(D10-DOUT): now reaches D11.3 (DIN)
- net Net-(D10-DOUT): now also D10.1 (DOUT)
- net Net-(D44-DOUT): now reaches D44.1 (DOUT), D45.3 (DIN)
- net Net-(D43-DOUT): now reaches D43.1 (DOUT), D44.3 (DIN)
- net Net-(D34-DOUT): now reaches D34.1 (DOUT), D35.3 (DIN)
- net Net-(D33-DOUT): now reaches D33.1 (DOUT), D34.3 (DIN)
- net Net-(D20-DOUT): now reaches D20.1 (DOUT)
- net Net-(D20-DOUT): now also D21.3 (DIN)
- net Net-(D45-DOUT): now reaches D45.1 (DOUT)
- net Net-(D45-DOUT): now also D46.3 (DIN)
- net Net-(D32-DOUT): now reaches D32.1 (DOUT), D33.3 (DIN)
- net Net-(D28-DOUT): now reaches D28.1 (DOUT), D29.3 (DIN)
- net Net-(D39-DOUT): now reaches D39.1 (DOUT), D40.3 (DIN)
- net Net-(D38-DOUT): now reaches D38.1 (DOUT), D39.3 (DIN)
- net Net-(D27-DOUT): now reaches D27.1 (DOUT), D28.3 (DIN)
- net Net-(D48-DOUT): now reaches D48.1 (DOUT), D49.3 (DIN)
- net Net-(D17-DOUT): now reaches D17.1 (DOUT), D18.3 (DIN)
- net Net-(D40-DOUT): now reaches D40.1 (DOUT)
- net Net-(D40-DOUT): now also D41.3 (DIN)
- net Net-(D12-DOUT): now reaches D12.1 (DOUT), D13.3 (DIN)
- net Net-(D42-DOUT): now reaches D42.1 (DOUT), D43.3 (DIN)
- net Net-(D41-DOUT): now reaches D41.1 (DOUT), D42.3 (DIN)
- net Net-(D31-DOUT): now reaches D31.1 (DOUT), D32.3 (DIN)
- net Net-(D23-DOUT): now reaches D23.1 (DOUT), D24.3 (DIN)
- net Net-(D22-DOUT): now reaches D22.1 (DOUT), D23.3 (DIN)
- net LEDA_DATA: now reaches D10.3 (DIN)
- net LEDA_DATA: now also J2.2
- net Net-(D16-DOUT): now reaches D16.1 (DOUT), D17.3 (DIN)
- net Net-(D37-DOUT): now reaches D37.1 (DOUT), D38.3 (DIN)
- net Net-(D26-DOUT): now reaches D26.1 (DOUT), D27.3 (DIN)
- net Net-(D15-DOUT): now reaches D15.1 (DOUT)
- net Net-(D15-DOUT): now also D16.3 (DIN)
- net Net-(D21-DOUT): now reaches D21.1 (DOUT), D22.3 (DIN)
- net LEDB_DATA: now reaches U1.7 (MTDO/GPIO7)
- net LEDB_DATA: now also D74.3 (DIN), J2.3
- net CC1: no longer names the net of R1.1
- net CC1: no longer J4.A5 (CC1)
- net CC2: no longer names the net of J4.B5 (CC2)
- net CC2: no longer R2.1
- net D+: no longer names the net of J4.A6 (D+), J4.B6 (D+)
- net D+: no longer U2.1 (I/O1)
- net D-: no longer names the net of J4.A7 (D-), J4.B7 (D-)
- net D-: no longer U2.3 (I/O2)
- net ESP_EN: no longer names the net of C4.1, D4.2 (A2), R7.2, SW1.2 (B)
- net ESP_EN: no longer U1.3 (EN/CHIP_PU)
- net GPIO3: no longer names the net of R8.2
- net GPIO3: no longer U1.26 (GPIO3/ADC1_CH3)
- net USB_D+: no longer names the net of U1.14 (GPIO13/USB_D+)
- net USB_D+: no longer U2.6 (I/O1)
- net USB_D-: no longer names the net of U1.13 (GPIO12/USB_D-)
- net USB_D-: no longer U2.4 (I/O2)
- new net Net-(D100-DOUT): D100.1 (DOUT), D101.3 (DIN)
- new net Net-(D101-DOUT): D101.1 (DOUT), D102.3 (DIN)
- new net Net-(D102-DOUT): D102.1 (DOUT), D103.3 (DIN)
- new net Net-(D103-DOUT): D103.1 (DOUT), D104.3 (DIN)
- new net Net-(D104-DOUT): D104.1 (DOUT), D105.3 (DIN)
- new net Net-(D105-DOUT): D105.1 (DOUT), D106.3 (DIN)
- new net Net-(D106-DOUT): D106.1 (DOUT), D107.3 (DIN)
- new net Net-(D107-DOUT): D107.1 (DOUT), D108.3 (DIN)
- new net Net-(D108-DOUT): D108.1 (DOUT), D109.3 (DIN)
- new net Net-(D109-DOUT): D109.1 (DOUT), D110.3 (DIN)
- new net Net-(D110-DOUT): D110.1 (DOUT), D111.3 (DIN)
- new net Net-(D111-DOUT): D111.1 (DOUT), D112.3 (DIN)
- new net Net-(D112-DOUT): D112.1 (DOUT), D113.3 (DIN)
- new net Net-(D113-DOUT): D113.1 (DOUT), D114.3 (DIN)
- new net Net-(D114-DOUT): D114.1 (DOUT), D115.3 (DIN)
- new net Net-(D115-DOUT): D115.1 (DOUT), D116.3 (DIN)
- new net Net-(D116-DOUT): D116.1 (DOUT), D117.3 (DIN)
- new net Net-(D117-DOUT): D117.1 (DOUT), D118.3 (DIN)
- new net Net-(D118-DOUT): D118.1 (DOUT), D119.3 (DIN)
- new net Net-(D119-DOUT): D119.1 (DOUT), D120.3 (DIN)
- new net Net-(D120-DOUT): D120.1 (DOUT), D121.3 (DIN)
- new net Net-(D121-DOUT): D121.1 (DOUT), D122.3 (DIN)
- new net Net-(D122-DOUT): D122.1 (DOUT), D123.3 (DIN)
- new net Net-(D123-DOUT): D123.1 (DOUT), D124.3 (DIN)
- new net Net-(D124-DOUT): D124.1 (DOUT), D125.3 (DIN)
- new net Net-(D125-DOUT): D125.1 (DOUT), D126.3 (DIN)
- new net Net-(D126-DOUT): D126.1 (DOUT), D127.3 (DIN)
- new net Net-(D127-DOUT): D127.1 (DOUT), D128.3 (DIN)
- new net Net-(D128-DOUT): D128.1 (DOUT), D129.3 (DIN)
- new net Net-(D129-DOUT): D129.1 (DOUT), D130.3 (DIN)
- new net Net-(D130-DOUT): D130.1 (DOUT), D131.3 (DIN)
- new net Net-(D131-DOUT): D131.1 (DOUT), D132.3 (DIN)
- new net Net-(D132-DOUT): D132.1 (DOUT), D133.3 (DIN)
- new net Net-(D133-DOUT): D133.1 (DOUT), D134.3 (DIN)
- new net Net-(D134-DOUT): D134.1 (DOUT), D135.3 (DIN)
- new net Net-(D135-DOUT): D135.1 (DOUT), D136.3 (DIN)
- new net Net-(D136-DOUT): D136.1 (DOUT), D137.3 (DIN)
- new net Net-(D137-DOUT): D137.1 (DOUT)
- new net Net-(D51-DOUT): D51.1 (DOUT), D52.3 (DIN)
- new net Net-(D52-DOUT): D52.1 (DOUT), D53.3 (DIN)
- new net Net-(D53-DOUT): D53.1 (DOUT), D54.3 (DIN)
- new net Net-(D54-DOUT): D54.1 (DOUT), D55.3 (DIN)
- new net Net-(D55-DOUT): D55.1 (DOUT), D56.3 (DIN)
- new net Net-(D56-DOUT): D56.1 (DOUT), D57.3 (DIN)
- new net Net-(D57-DOUT): D57.1 (DOUT), D58.3 (DIN)
- new net Net-(D58-DOUT): D58.1 (DOUT), D59.3 (DIN)
- new net Net-(D59-DOUT): D59.1 (DOUT), D60.3 (DIN)
- new net Net-(D60-DOUT): D60.1 (DOUT), D61.3 (DIN)
- new net Net-(D61-DOUT): D61.1 (DOUT), D62.3 (DIN)
- new net Net-(D62-DOUT): D62.1 (DOUT), D63.3 (DIN)
- new net Net-(D63-DOUT): D63.1 (DOUT), D64.3 (DIN)
- new net Net-(D64-DOUT): D64.1 (DOUT), D65.3 (DIN)
- new net Net-(D65-DOUT): D65.1 (DOUT), D66.3 (DIN)
- new net Net-(D66-DOUT): D66.1 (DOUT), D67.3 (DIN)
- new net Net-(D67-DOUT): D67.1 (DOUT), D68.3 (DIN)
- new net Net-(D68-DOUT): D68.1 (DOUT), D69.3 (DIN)
- new net Net-(D69-DOUT): D69.1 (DOUT), D70.3 (DIN)
- new net Net-(D70-DOUT): D70.1 (DOUT), D71.3 (DIN)
- new net Net-(D71-DOUT): D71.1 (DOUT), D72.3 (DIN)
- new net Net-(D72-DOUT): D72.1 (DOUT), D73.3 (DIN)
- new net Net-(D73-DOUT): D73.1 (DOUT)
- new net Net-(D74-DOUT): D74.1 (DOUT), D75.3 (DIN)
- new net Net-(D75-DOUT): D75.1 (DOUT), D76.3 (DIN)
- new net Net-(D76-DOUT): D76.1 (DOUT), D77.3 (DIN)
- new net Net-(D77-DOUT): D77.1 (DOUT), D78.3 (DIN)
- new net Net-(D78-DOUT): D78.1 (DOUT), D79.3 (DIN)
- new net Net-(D79-DOUT): D79.1 (DOUT), D80.3 (DIN)
- new net Net-(D80-DOUT): D80.1 (DOUT), D81.3 (DIN)
- new net Net-(D81-DOUT): D81.1 (DOUT), D82.3 (DIN)
- new net Net-(D82-DOUT): D82.1 (DOUT), D83.3 (DIN)
- new net Net-(D83-DOUT): D83.1 (DOUT), D84.3 (DIN)
- new net Net-(D84-DOUT): D84.1 (DOUT), D85.3 (DIN)
- new net Net-(D85-DOUT): D85.1 (DOUT), D86.3 (DIN)
- new net Net-(D86-DOUT): D86.1 (DOUT), D87.3 (DIN)
- new net Net-(D87-DOUT): D87.1 (DOUT), D88.3 (DIN)
- new net Net-(D88-DOUT): D88.1 (DOUT), D89.3 (DIN)
- new net Net-(D89-DOUT): D89.1 (DOUT), D90.3 (DIN)
- new net Net-(D90-DOUT): D90.1 (DOUT), D91.3 (DIN)
- new net Net-(D91-DOUT): D91.1 (DOUT), D92.3 (DIN)
- new net Net-(D92-DOUT): D92.1 (DOUT), D93.3 (DIN)
- new net Net-(D93-DOUT): D93.1 (DOUT), D94.3 (DIN)
- new net Net-(D94-DOUT): D94.1 (DOUT), D95.3 (DIN)
- new net Net-(D95-DOUT): D95.1 (DOUT), D96.3 (DIN)
- new net Net-(D96-DOUT): D96.1 (DOUT), D97.3 (DIN)
- new net Net-(D97-DOUT): D97.1 (DOUT), D98.3 (DIN)
- new net Net-(D98-DOUT): D98.1 (DOUT), D99.3 (DIN)
- new net Net-(D99-DOUT): D100.3 (DIN), D99.1 (DOUT)
- no-connect marks 2 -> 0
Other:
- note removed: "POWER REGULATOR"
- note removed: "RESET BUTTON"
- note removed: "USB-C"
- title: ESP32-S3 -> ESP32-C6 LED Matrix (8x8 double-sided, 128 LEDs)
